File: pixdog.kicad_sch (KiCad schematic)
At the start: 0 parts

Commit message: updates
Other:
- sheet Servo ports: added +5V_Internal, +5V_Servo, I2C_SCL, I2C_SDA; removed none
Changed lines of the file:
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@@
 	)
 	(sheet
-		(at 45.72 73.66)
-		(size 48.26 34.29)
+		(at 54.61 83.82)
+		(size 27.94 10.16)
 		(exclude_from_sim no)
 		(in_bom yes)
@@
 		)
 		(property "Sheetname" "Servo"
-			(at 45.72 72.9484 0)
+			(at 54.61 83.1084 0)
 			(show_name no)
 			(do_not_autoplace no)
@@
 		)
 		(property "Sheetfile" "servo.kicad_sch"
-			(at 45.72 108.5346 0)
+			(at 54.61 94.5646 0)
 			(show_name no)
 			(do_not_autoplace no)
@@
 			)
 		)
+		(pin "+5V_Internal" input
+			(at 54.61 87.63 180)
+			(effects
+				(font
+					(size 1.27 1.27)
+				)
+				(justify left)
+			)
+		)
+		(pin "+5V_Servo" input
+			(at 54.61 90.17 180)
+			(effects
+				(font
+					(size 1.27 1.27)
+				)
+				(justify left)
+			)
+		)
+		(pin "I2C_SCL" bidirectional
+			(at 82.55 87.63 0)
+			(effects
+				(font
+					(size 1.27 1.27)
+				)
+				(justify right)
+			)
+		)
+		(pin "I2C_SDA" bidirectional
+			(at 82.55 90.17 0)
+			(effects
+				(font
+					(size 1.27 1.27)
+				)
+				(justify right)
+			)
+		)
