File: servo.kicad_sch (KiCad schematic)
At the start: 0 parts

Commit message: updates
Parts:
- added C1: 10uF, symbol Device:C_Small
- added D1, D2: Green, symbol Device:LED_Small
- added J10, J11, J12, J13, J14, J15, J16, J17, J18, J19, J20, J21, J3, J7, J8, J9: Conn_01x03, symbol Connector_Generic:Conn_01x03
- added R1, R2: 10k, symbol Device:R_Small
- added R13, R14, R15, R16, R17, R18, R19, R20, R21, R22, R23, R24, R25, R26, R3, R4, R5, R6: 470, symbol Device:R_Small
- added U2: PCA9685PW, Package_SO:TSSOP-28_4.4x9.7mm_P0.65mm, symbol Driver_LED:PCA9685PW
Connections:
- new net: J21.1 (Pin_1), R26.2
- new net: J13.1 (Pin_1), R18.2
- new net: J11.1 (Pin_1), R16.2
- new net: J14.1 (Pin_1), R19.2
- new net: J12.1 (Pin_1), R17.2
- new net: J19.1 (Pin_1), R24.2
- new net: J15.1 (Pin_1), R20.2
- new net: J8.1 (Pin_1), R13.2
- new net: D2.1 (K), R4.1
- new net: J9.1 (Pin_1), R14.2
- new net: D1.1 (K), R3.1
- new net: J18.1 (Pin_1), R23.2
- new net: J16.1 (Pin_1), R21.2
- new net: J7.1 (Pin_1), R6.2
- new net: J17.1 (Pin_1), R22.2
- new net: J10.1 (Pin_1), R15.2
- new net: J20.1 (Pin_1), R25.2
- new net: J3.1 (Pin_1), R5.2
- new net +5V_Internal: C1.1, D1.2 (A), R2.2, U2.1 (A0), U2.28 (VDD), U2.3 (A2), U2.5 (A4)
- new net +5V_Servo: D2.2 (A), J10.2 (Pin_2), J11.2 (Pin_2), J12.2 (Pin_2), J13.2 (Pin_2), J14.2 (Pin_2), J15.2 (Pin_2), J16.2 (Pin_2), J17.2 (Pin_2), J18.2 (Pin_2), J19.2 (Pin_2), J20.2 (Pin_2), J21.2 (Pin_2), J3.2 (Pin_2), J7.2 (Pin_2), J8.2 (Pin_2), J9.2 (Pin_2)
- new net GND: C1.2, J10.3 (Pin_3), J11.3 (Pin_3), J12.3 (Pin_3), J13.3 (Pin_3), J14.3 (Pin_3), J15.3 (Pin_3), J16.3 (Pin_3), J17.3 (Pin_3), J18.3 (Pin_3), J19.3 (Pin_3), J20.3 (Pin_3), J21.3 (Pin_3), J3.3 (Pin_3), J7.3 (Pin_3), J8.3 (Pin_3), J9.3 (Pin_3), R1.1, R2.1, R3.2, R4.2, U2.14 (VSS), U2.2 (A1), U2.24 (A5), U2.25 (EXTCLK), U2.4 (A3)
- new net I2C_SCL: U2.26 (SCL)
- new net I2C_SDA: U2.27 (SDA)
- new net PWM0: R5.1, U2.6 (LED0)
- new net PWM1: R6.1, U2.7 (LED1)
- new net PWM10: R21.1, U2.17 (LED10)
- new net PWM11: R22.1, U2.18 (LED11)
- new net PWM12: R23.1, U2.19 (LED12)
- new net PWM13: R24.1, U2.20 (LED13)
- new net PWM14: R25.1, U2.21 (LED14)
- new net PWM15: R26.1, U2.22 (LED15)
- new net PWM2: R13.1, U2.8 (LED2)
- new net PWM3: R14.1, U2.9 (LED3)
- new net PWM4: R15.1, U2.10 (LED4)
- new net PWM5: R16.1, U2.11 (LED5)
- new net PWM6: R17.1, U2.12 (LED6)
- new net PWM7: R18.1, U2.13 (LED7)
- new net PWM8: R19.1, U2.15 (LED8)
- new net PWM9: R20.1, U2.16 (LED9)
- new net nOE: R1.2, U2.23 (~{OE})
Other:
- note added: "Main Servo Connection"
- note added: "Power Status LEDs"
- note added: "Servo Driver (I2C addr 0x1010101)"
- note added: "Spare Servo Connection"
